File: Balanca2.kicad_sch (KiCad schematic)
At the start: 39 parts, among them J1 Conn_01x03_Pin, J2 Conn_01x03_Pin, J3 Conn_01x03_Pin, J4 Conn_01x03_Pin, J5 Conn_01x03_Pin, J6 Conn_01x03, J7 Conn_01x05, Q1 BC547, Q2 BC557, U1 TL084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

Commit message: Ajuste inicial da versao 2
Parts:
- removed R10: 100k, Resistor_THT:R_Axial_DIN0207_L6.3mm_D2.5mm_P2.54mm_Vertical, symbol Device:R
- removed R11: 100k, Resistor_THT:R_Axial_DIN0204_L3.6mm_D1.6mm_P2.54mm_Vertical, symbol Device:R
- removed R5, R7: 33k, Resistor_THT:R_Axial_DIN0207_L6.3mm_D2.5mm_P2.54mm_Vertical, symbol Device:R
- removed R6: 330, Resistor_THT:R_Axial_DIN0207_L6.3mm_D2.5mm_P10.16mm_Horizontal, symbol Device:R
- removed R8: 10k, Resistor_THT:R_Axial_DIN0207_L6.3mm_D2.5mm_P10.16mm_Horizontal, symbol Device:R
- removed R9: 10k, Resistor_THT:R_Axial_DIN0207_L6.3mm_D2.5mm_P15.24mm_Horizontal, symbol Device:R
- removed U1: TL084, Package_DIP:DIP-14_W7.62mm, symbol Amplifier_Operational:TL084
- removed unit 3 of U3
- added U1: TL082, symbol Amplifier_Operational:TL082
- added U2: INA128, Package_DIP:DIP-8_W7.62mm, symbol Amplifier_Instrumentation:INA128
- added U8: LM393, symbol Comparator:LM393
- RV3: value 10k -> 50k
Connections:
- net +15V: now also U2.7 (V+)
- net +5V: now also U1.8 (V+)
- net -15V: now also U2.4 (V-)
- net -5V: now also U1.4 (V-)
- net AC: now also U1.3 (+)
- net CelulaCargaAlimentacaoV+: now also U1.2 (-)
- net SaidaPrimeiroEstagio: now also U2.6
- net SinalSaida+: now also U2.3 (+)
- net SinalSaida-: now also U2.2 (-)
- net at Q1.2 (B), Q2.2 (B): now also U1.1
- net at RV3.1: now also U2.8 (Rg)
- net at RV3.2, RV3.3: now also U2.1 (Rg)
Other:
- moved on the sheet: JP5, JP6, JP7, RV3, U7C

Commit message: Mudança da placa v2
Parts:
- removed JP1: Jumper_2_Bridged, TestPoint:TestPoint_Bridge_Pitch5.08mm_Drill0.7mm, symbol Jumper:Jumper_2_Bridged
- removed U3: TL082, Package_DIP:DIP-8_W7.62mm, symbol Amplifier_Operational:TL082
- U1, U8: footprint (none) -> Package_DIP:DIP-8_W7.62mm
Connections:
- net +15V: now also U1.8 (V+)
- net +5V: now also U8.8 (V+); no longer U1.8 (V+)
- net -15V: now also U1.4 (V-)
- net -5V: now also U8.4 (V-); no longer U1.4 (V-)
- net AC: now also U1.5 (+); no longer U1.3 (+)
- net CelulaCargaAlimentacaoV+: now also J6.3 (Pin_3), U1.6 (-), U8.3 (+), U8.6 (-); no longer J6.1 (Pin_1), U1.2 (-)
- net Controle1: now also U8.1
- net Controle2: now also U8.7
- net GND: now also J6.1 (Pin_1), U2.5 (Ref), U6.8, U8.2 (-), U8.5 (+); no longer J6.3 (Pin_3), U6.10
- net SaidaPrimeiroEstagio: now also U6.10; no longer U6.8
- net at Q1.2 (B), Q2.2 (B): now also U1.7; no longer U1.1
- no-connect marks 7 -> 10
Other:
- moved on the sheet: U8A, U8B, U8C

Commit message: Atualizacao da versao 3
Parts:
- added C10, C11, C12, C13, C14, C15, C6, C7, C8, C9: 100n, Capacitor_THT:C_Disc_D5.0mm_W2.5mm_P2.50mm, symbol Device:C
- added R5, R6: 10k, Resistor_THT:R_Axial_DIN0207_L6.3mm_D2.5mm_P10.16mm_Horizontal, symbol Device:R
- C2, C3: value C_Polarized -> 1u
- R3: value 22k -> 47k
- RV3: value 50k -> 10K
Connections:
- net +15V: now also C10.1, C12.2, C7.2
- net +5V: now also C14.2, C8.2, R5.2, R6.2
- net -15V: now also C11.1, C13.2, C6.2
- net -5V: now also C15.2, C9.2
- net Controle1: now also R6.1
- net Controle2: now also R5.1
- net GND: now also C10.2, C11.2, C12.1, C13.1, C14.1, C15.1, C6.1, C7.1, C8.1, C9.1
- net at RV3.2, RV3.3: now also U2.8 (Rg); no longer U2.1 (Rg)
- net at RV3.1: now also U2.1 (Rg); no longer U2.8 (Rg)
Other:
- note added: "ALIMENTAÇÃO"
- note added: "ALIMENTAÇÃO CELULA DE CARGA + CONECTORES"
- note added: "AMPLIFICADOR DE GANHO 4,7"
- note added: "AMPLIFICADOR DE INSTRUMENTAÇÃO - GANHO DE 1 A 10000"
- note added: "ZERO CROSSING/CONTROLE DAS CHAVES"
- note removed: "AMPLIFICADOR DE GANHO 2,2"
- note removed: "AMPLIFICADOR DE INSTRUMENTAÇÃO - GANHO DE 163 A 4400"
- note removed: "CONECTORES"
- moved on the sheet: C1, D1, D2, J1, J2, J3, J4, J5, J6, J7, JP5, JP6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

Commit message: Atualizacao de esquematico da placa 3
Parts:
- removed D1, D2: 1N4007, Diode_THT:D_DO-41_SOD81_P10.16mm_Horizontal, symbol Diode:1N4007
- added C16: 33p, Capacitor_THT:C_Disc_D5.0mm_W2.5mm_P2.50mm, symbol Device:C
- added C17: 4,7u, Capacitor_THT:CP_Radial_D5.0mm_P2.50mm, symbol Device:C_Polarized
- added D3, D4: 1N4007, Diode_THT:D_DO-41_SOD81_P10.16mm_Horizontal, symbol Diode:1N4007
- added R10, R11: 100k, Resistor_THT:R_Axial_DIN0207_L6.3mm_D2.5mm_P2.54mm_Vertical, symbol Device:R
- added R12: 10k, Resistor_THT:R_Axial_DIN0207_L6.3mm_D2.5mm_P10.16mm_Horizontal, symbol Device:R
- added R7, R8: 330, Resistor_THT:R_Axial_DIN0207_L6.3mm_D2.5mm_P10.16mm_Horizontal, symbol Device:R
- added R9: 33, Resistor_THT:R_Axial_DIN0207_L6.3mm_D2.5mm_P10.16mm_Horizontal, symbol Device:R
- C1: value 50n -> 470n
Connections:
- net +15V: now also C14.2, U4.1 (VI), U8.8 (V+), D3.1 (K), R11.2, R7.2; no longer J3.1 (Pin_1), J3.2 (Pin_2), J3.3 (Pin_3), Q1.1 (C), RV1.3
- net +5V: no longer C14.2, U8.8 (V+)
- net -15V: now also U5.2 (VI), D4.2 (A), R10.1, R8.1; no longer J2.1 (Pin_1), J2.2 (Pin_2), J2.3 (Pin_3), Q2.1 (C), RV1.1
- net -5V: now also U6.13, U6.5
- net CelulaCargaAlimentacaoV+: now also C16.2, R9.2; no longer Q1.3 (E), Q2.3 (E)
- net GND: now also U1.3 (+), U6.1, U6.2, U6.3, U6.4, C16.1, C17.2; no longer U6.13
- net at C1.1, U7.2 (-): now also R12.2; no longer R1.2, R3.1
- net at U1.1: now also U1.2 (-)
- new net: R10.2, RV1.1
- new net: R11.1, RV1.3
- new net: Q2.1 (C), R8.2
- new net: Q1.3 (E), Q2.3 (E), R9.1
- new net: C17.1, R1.2, R12.1, R3.1
- new net: Q1.1 (C), R7.1
- new net Entrada+15V: D3.2 (A), J3.1 (Pin_1), J3.2 (Pin_2), J3.3 (Pin_3)
- new net Entrada-15V: D4.1 (K), J2.1 (Pin_1), J2.2 (Pin_2), J2.3 (Pin_3)
- no-connect marks 10 -> 2
Other:
- note added: "CAPACITORES E CONEXOES"
- note added: "DEMODULADOR"
- note removed: "CURTOS"
- title: (none) -> Balanca AC
- moved on the sheet: C10, C11, C12, C13, C14, C15, C2, C3, C4, C5, C6, C7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

Commit message: Inicio do Roteamento
Other:
- moved on the sheet: C6, C7, JP5, JP6, JP7, RV3, U2

Commit message: Atualizacao de footprints
Parts:
- R5: footprint Resistor_THT:R_Axial_DIN0207_L6.3mm_D2.5mm_P10.16mm_Horizontal -> Resistor_THT:R_Axial_DIN0204_L3.6mm_D1.6mm_P5.08mm_Vertical
Connections:
- net SaídaBuffer: now reaches Q1.2 (B), Q2.2 (B), U1.7
Changed lines of the file:
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@@
 		)
 	)
+	(label "SaídaBuffer"
+		(at 69.85 129.54 180)
+		(effects
+			(font
+				(size 1.27 1.27)
+			)
+			(justify right bottom)
+		)
+	)
 	(label "SaidaDemodulada"
 		(at 33.02 232.41 180)
@@
 			)
 		)
-		(property "Footprint" "Resistor_THT:R_Axial_DIN0207_L6.3mm_D2.5mm_P10.16mm_Horizontal"
+		(property "Footprint" "Resistor_THT:R_Axial_DIN0204_L3.6mm_D1.6mm_P5.08mm_Vertical"
 			(at 194.818 217.17 90)
 			(hide yes)

Commit message: Roteamento iniciado, falta verificar erros
Parts:
- R10, R11: footprint Resistor_THT:R_Axial_DIN0207_L6.3mm_D2.5mm_P2.54mm_Vertical -> Resistor_THT:R_Axial_DIN0207_L6.3mm_D2.5mm_P10.16mm_Horizontal
- R8: footprint Resistor_THT:R_Axial_DIN0207_L6.3mm_D2.5mm_P10.16mm_Horizontal -> Resistor_THT:R_Axial_DIN0207_L6.3mm_D2.5mm_P5.08mm_Vertical
Connections:
- net +15V: now also R10.2; no longer R11.2
- net -15V: now also R11.1; no longer R10.1
- net at RV1.1: now also R10.1; no longer R10.2
- net at RV1.3: now also R11.2; no longer R11.1
Other:
- moved on the sheet: R10, R11, RV1
Changed lines of the file:
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@@
 	(wire
 		(pts
-			(xy 92.71 203.2) (xy 91.44 203.2)
+			(xy 149.86 119.38) (xy 152.4 119.38)
 		)
 		(stroke
@@
 	(wire
 		(pts
-			(xy 149.86 119.38) (xy 152.4 119.38)
+			(xy 162.56 44.45) (xy 163.83 44.45)
 		)
 		(stroke
@@
 	(wire
 		(pts
-			(xy 162.56 44.45) (xy 163.83 44.45)
+			(xy 25.4 60.96) (xy 24.13 60.96)
 		)
 		(stroke
@@
 	(wire
 		(pts
-			(xy 25.4 60.96) (xy 24.13 60.96)
+			(xy 31.75 160.02) (xy 30.48 160.02)
 		)
 		(stroke
@@
 	(wire
 		(pts
-			(xy 31.75 160.02) (xy 30.48 160.02)
+			(xy 74.93 234.95) (xy 71.12 234.95)
 		)
 		(stroke
@@
 	(wire
 		(pts
-			(xy 74.93 234.95) (xy 71.12 234.95)
+			(xy 91.44 203.2) (xy 92.71 203.2)
 		)
 		(stroke
@@
 	(symbol
 		(lib_id "Device:R_Potentiometer")
-		(at 96.52 203.2 90)
-		(mirror x)
+		(at 96.52 203.2 270)
 		(unit 1)
 		(body_style 1)
@@
 		(dnp no)
 		(property "Reference" "RV1"
-			(at 95.2499 200.66 0)
+			(at 97.7901 200.66 0)
 			(show_name no)
 			(do_not_autoplace no)
@@
 		)
 		(property "Value" "10k"
-			(at 97.7899 200.66 0)
+			(at 95.2501 200.66 0)
 			(show_name no)
 			(do_not_autoplace no)
@@
 	(symbol
 		(lib_id "Device:R")
-		(at 105.41 203.2 90)
+		(at 87.63 203.2 90)
 		(unit 1)
 		(body_style 1)
@@
 		(fields_autoplaced yes)
 		(property "Reference" "R11"
-			(at 106.6801 205.74 0)
+			(at 88.9001 205.74 0)
 			(show_name no)
 			(do_not_autoplace no)
@@
 		)
 		(property "Value" "100k"
-			(at 104.1401 205.74 0)
+			(at 86.3601 205.74 0)
 			(show_name no)
 			(do_not_autoplace no)
@@
 			)
 		)
-		(property "Footprint" "Resistor_THT:R_Axial_DIN0207_L6.3mm_D2.5mm_P2.54mm_Vertical"
-			(at 105.41 204.978 90)
+		(property "Footprint" "Resistor_THT:R_Axial_DIN0207_L6.3mm_D2.5mm_P10.16mm_Horizontal"
+			(at 87.63 204.978 90)
 			(hide yes)
 			(show_name no)
@@
 		)
 		(property "Datasheet" ""
-			(at 105.41 203.2 0)
+			(at 87.63 203.2 0)
 			(hide yes)
 			(show_name no)
@@
 		)
 		(property "Description" "Resistor"
-			(at 105.41 203.2 0)
+			(at 87.63 203.2 0)
 			(hide yes)
 			(show_name no)
@@
 			)
 		)
-		(property "Footprint" "Resistor_THT:R_Axial_DIN0207_L6.3mm_D2.5mm_P10.16mm_Horizontal"
+		(property "Footprint" "Resistor_THT:R_Axial_DIN0207_L6.3mm_D2.5mm_P5.08mm_Vertical"
 			(at 74.93 140.208 90)
 			(hide yes)
@@
 	(symbol
 		(lib_id "Device:R")
-		(at 87.63 203.2 90)
+		(at 105.41 203.2 90)
 		(unit 1)
 		(body_style 1)
@@
 		(fields_autoplaced yes)
 		(property "Reference" "R10"
-			(at 88.9001 205.74 0)
+			(at 106.6801 205.74 0)
 			(show_name no)
 			(do_not_autoplace no)
@@
 		)
 		(property "Value" "100k"
-			(at 86.3601 205.74 0)
+			(at 104.1401 205.74 0)
 			(show_name no)
 			(do_not_autoplace no)
@@
 			)
 		)
-		(property "Footprint" "Resistor_THT:R_Axial_DIN0207_L6.3mm_D2.5mm_P2.54mm_Vertical"
-			(at 87.63 204.978 90)
+		(property "Footprint" "Resistor_THT:R_Axial_DIN0207_L6.3mm_D2.5mm_P10.16mm_Horizontal"
+			(at 105.41 204.978 90)
 			(hide yes)
 			(show_name no)
@@
 		)
 		(property "Datasheet" ""
-			(at 87.63 203.2 0)
+			(at 105.41 203.2 0)
 			(hide yes)
 			(show_name no)
@@
 		)
 		(property "Description" "Resistor"
-			(at 87.63 203.2 0)
+			(at 105.41 203.2 0)
 			(hide yes)
 			(show_name no)

Commit message: Alteracoes de footprint e melhorias de trilhas
Parts:
- removed C4: C_Polarized, Capacitor_THT:CP_Radial_D5.0mm_P2.50mm, symbol Device:C_Polarized
- removed C8: 100n, Capacitor_THT:C_Disc_D5.0mm_W2.5mm_P2.50mm, symbol Device:C
- removed JP7: Jumper_2_Bridged, TestPoint:TestPoint_Bridge_Pitch5.08mm_Drill0.7mm, symbol Jumper:Jumper_2_Bridged
- added C18: 100n, Capacitor_THT:C_Disc_D5.0mm_W2.5mm_P2.50mm, symbol Device:C
- added JP10: Jumper_2_Bridged, Library:TestPoint_Bridge_Pitch7.62mm_Drill1.3mm, symbol Jumper:Jumper_2_Bridged
- added JP8: Jumper_2_Bridged, Library:TestPoint_Bridge_Pitch6.35mm_Drill1.3mm, symbol Jumper:Jumper_2_Bridged
- added JP9: Jumper_2_Bridged, Library:TestPoint_Bridge_Pitch5.08mm_Drill1.3mm, symbol Jumper:Jumper_2_Bridged
- R10, R11, R7: footprint Resistor_THT:R_Axial_DIN0207_L6.3mm_D2.5mm_P10.16mm_Horizontal -> Resistor_THT:R_Axial_DIN0207_L6.3mm_D2.5mm_P15.24mm_Horizontal
Connections:
- net +15V: now also JP9.1 (A); no longer U8.8 (V+)
- net +5V: now also C18.1
- net CelulaCargaAlimentacaoV+: now also JP8.1 (A); no longer U8.3 (+), U8.6 (-)
- net GND: now also C18.2
- net SaidaPrimeiroEstagio: now also JP10.2 (B); no longer R4.1
- new net: JP9.2 (B), U8.8 (V+)
- new net: JP8.2 (B), U8.3 (+), U8.6 (-)
- new net SaidaPrimeiroEstagioA: JP10.1 (A), R4.1
Other:
- moved on the sheet: C14
