File: Balanca2.kicad_sch (KiCad schematic)
At the start: 53 parts, among them J1 Conn_01x03_Pin, J2 Conn_01x03_Pin, J3 Conn_01x03_Pin, J4 Conn_01x03_Pin, J5 Conn_01x03_Pin, J6 Conn_01x03, J7 Conn_01x05, Q1 BC547, Q2 BC557, U1 TL082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

Commit message: Finalizada Versao 3
Parts:
- JP8: footprint Library:TestPoint_Bridge_Pitch6.35mm_Drill1.3mm -> Library:TestPoint_Bridge_Pitch7.62mm_Drill1.3mm
- R10, R11: footprint Resistor_THT:R_Axial_DIN0207_L6.3mm_D2.5mm_P15.24mm_Horizontal -> Resistor_THT:R_Axial_DIN0207_L6.3mm_D2.5mm_P10.16mm_Horizontal
Connections:
- net CelulaCargaAlimentacaoV+: now also JP8.2 (B), U8.3 (+), U8.6 (-)
Changed lines of the file:
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@@
 	)
 	(junction
+		(at 153.67 226.06)
+		(diameter 0)
+		(color 0 0 0 0)
+	)
+	(junction
 		(at 213.36 67.31)
 		(diameter 0)
@@
 	)
 	(junction
+		(at 165.1 231.14)
+		(diameter 0)
+		(color 0 0 0 0)
+	)
+	(junction
 		(at 69.85 121.92)
 		(diameter 0)
@@
 	(wire
 		(pts
-			(xy 165.1 226.06) (xy 165.1 237.49)
+			(xy 165.1 226.06) (xy 165.1 231.14)
 		)
 		(stroke
@@
 	(wire
 		(pts
+			(xy 153.67 226.06) (xy 153.67 231.14)
+		)
+		(stroke
+			(width 0)
+			(type default)
+		)
+	)
+	(wire
+		(pts
 			(xy 81.28 123.19) (xy 78.74 123.19)
 		)
@@
 	(wire
 		(pts
+			(xy 153.67 231.14) (xy 165.1 231.14)
+		)
+		(stroke
+			(width 0)
+			(type default)
+		)
+	)
+	(wire
+		(pts
 			(xy 26.67 121.92) (xy 26.67 124.46)
 		)
@@
 	(wire
 		(pts
+			(xy 165.1 231.14) (xy 165.1 237.49)
+		)
+		(stroke
+			(width 0)
+			(type default)
+		)
+	)
+	(wire
+		(pts
 			(xy 251.46 35.56) (xy 261.62 35.56)
 		)
@@
 		)
 	)
+	(label "CelulaCargaAlimentacaoV+x"
+		(at 165.1 237.49 180)
+		(effects
+			(font
+				(size 1.27 1.27)
+			)
+			(justify right bottom)
+		)
+	)
 	(label "Sense-"
 		(at 72.39 151.13 0)
@@
 			)
 		)
-		(property "Footprint" "Library:TestPoint_Bridge_Pitch6.35mm_Drill1.3mm"
+		(property "Footprint" "Library:TestPoint_Bridge_Pitch7.62mm_Drill1.3mm"
 			(at 158.75 226.06 0)
 			(hide yes)
@@
 			)
 		)
-		(property "Footprint" "Resistor_THT:R_Axial_DIN0207_L6.3mm_D2.5mm_P15.24mm_Horizontal"
+		(property "Footprint" "Resistor_THT:R_Axial_DIN0207_L6.3mm_D2.5mm_P10.16mm_Horizontal"
 			(at 87.63 204.978 90)
 			(hide yes)
@@
 			)
 		)
-		(property "Footprint" "Resistor_THT:R_Axial_DIN0207_L6.3mm_D2.5mm_P15.24mm_Horizontal"
+		(property "Footprint" "Resistor_THT:R_Axial_DIN0207_L6.3mm_D2.5mm_P10.16mm_Horizontal"
 			(at 105.41 204.978 90)
 			(hide yes)
